File: electrical/electrical.kicad_pcb (KiCad board)
At the start: 2 copper layers, 112.8 x 98.2 mm, 58 parts, among them J1 Raspberry Pi GPIO, J2 Conn_01x05_Pin, J3 Load_cell, J4 PIR_sensor, J9 Water_sensor, K1 RAYEX-L90, M1 Milk_powder, M2 Instant_coffee, M3 Sugar, M4 Motor_DC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

Commit message: added adjustment
Parts:
- J2: value Conn_01x05_Pin -> Touch screen connector
- e1: moved to B.Cu
Connections:
- net /Untitled Sheet2/OUT1 renamed /IR 2/OUT1
- net /Untitled Sheet2/OUT2 renamed /IR 2/OUT2
- J1 pad 35: GPIO19 -> /COFFEE
- J1 pad 37: GPIO26 -> /SUGAR
- R17 pad 1: /Untitled Sheet1/OUT1 -> /COFFEE
- R18 pad 1: /Untitled Sheet1/OUT2 -> /SUGAR
- R4 pad 1: unconnected-(R4-Pad1) -> GPIO4
- R9 pad 2: unconnected-(R9-Pad2) -> GPIO17
- U6 pad 1: /Untitled Sheet1/OUT1 -> /COFFEE
- U6 pad 7: /Untitled Sheet1/OUT2 -> /SUGAR
Routing:
- net GPIO14: track 49.4 -> 73.6 mm, vias 0 -> 2
- net GPIO17: track 0.00 -> 12.4 mm
- net GPIO4: track 0.00 -> 12.0 mm
- net /Untitled Sheet1/OUT1: track 10.0 -> 0.00 mm
- net /COFFEE: track 0.00 -> 10.0 mm
- net GPIO18: track 73.1 -> 81.4 mm, vias 0 -> 2
- net /Untitled Sheet1/OUT2: track 5.40 -> 0.00 mm
- net /SUGAR: track 0.00 -> 5.40 mm
