File: electrical/_autosave-electrical.kicad_pcb (KiCad board)
At the start: 2 copper layers, 112.8 x 98.2 mm, 58 parts, among them J1 Raspberry Pi GPIO, J2 Touch screen connector, J3 Load_cell, J4 PIR_sensor, J9 Water_sensor, K1 RAYEX-L90, M1 Milk_powder, M2 Instant_coffee, M3 Sugar, M4 Motor_DC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

Commit message: added scrolling feature
Parts:
- moved Q4 15.1 mm to (148.3, 95.4)
- moved R8 3.36 mm to (139.2, 103.5)
- moved R9 2.06 mm to (144.2, 101.2), turned to 180 degrees
Routing:
- net Net-(D1-A): track 45.9 -> 12.0 mm
- net GPIO22: track 16.5 -> 0.00 mm
- net Net-(D6-A): track 9.43 -> 13.8 mm
- net Net-(Q4-B): track 3.79 -> 0.00 mm
- net GPIO27: track 19.4 -> 21.9 mm
- net +12V: track 309.5 -> 307.3 mm
- net Net-(Q1-B): track 4.02 -> 4.83 mm
Changed lines of the file:
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@@
 	(footprint "Package_TO_SOT_THT:TO-92_Inline_Wide"
 		(layer "F.Cu")
-		(at 161.75 102.25 180)
+		(at 148.29 95.39 180)
 		(descr "TO-92 leads in-line, wide, drill 0.75mm (see NXP sot054_po.pdf)")
 		(tags "to-92 sc-43 sc-43a sot54 PA33 transistor")
@@
 	(footprint "Resistor_SMD:R_1206_3216Metric_Pad1.30x1.75mm_HandSolder"
 		(layer "B.Cu")
-		(at 146.25 101.05 90)
+		(at 144.2 101.25 180)
 		(descr "Resistor SMD 1206 (3216 Metric), square (rectangular) end terminal, IPC_7351 nominal with elongated pad for handsoldering. (Body size source: IPC-SM-782 page 72, https://www.pcb-3d.com/wordpress/wp-content/uploads/ipc-sm-782a_amendment_1_and_2.pdf), generated with kicad-footprint-generator")
 		(tags "resistor handsolder")
 		(property "Reference" "R9"
-			(at 0 1.82 90)
+			(at 0 1.82 360)
 			(layer "B.SilkS")
 			(effects
@@
 		)
 		(property "Value" "10K"
-			(at 0 -1.82 90)
+			(at 0 -1.82 360)
 			(layer "B.Fab")
 			(effects
@@
 		)
 		(property "Footprint" "Resistor_SMD:R_1206_3216Metric_Pad1.30x1.75mm_HandSolder"
-			(at 0 0 -90)
+			(at 0 0 0)
 			(unlocked yes)
 			(layer "B.Fab")
@@
 		)
 		(property "Datasheet" ""
-			(at 0 0 -90)
+			(at 0 0 0)
 			(unlocked yes)
 			(layer "B.Fab")
@@
 		)
 		(property "Description" "Resistor"
-			(at 0 0 -90)
+			(at 0 0 0)
 			(unlocked yes)
 			(layer "B.Fab")
@@
 		(attr smd)
 		(fp_line
-			(start 0.727064 -0.91)
-			(end -0.727064 -0.91)
+			(start 0.727064 0.91)
+			(end -0.727064 0.91)
 			(stroke
 				(width 0.12)
@@
 		)
 		(fp_line
-			(start 0.727064 0.91)
-			(end -0.727064 0.91)
+			(start 0.727064 -0.91)
+			(end -0.727064 -0.91)
 			(stroke
 				(width 0.12)
@@
 		)
 		(fp_line
-			(start 2.45 -1.12)
-			(end 2.45 1.12)
+			(start 2.45 1.12)
+			(end -2.45 1.12)
 			(stroke
 				(width 0.05)
@@
 		)
 		(fp_line
-			(start -2.45 -1.12)
-			(end 2.45 -1.12)
+			(start 2.45 -1.12)
+			(end 2.45 1.12)
 			(stroke
 				(width 0.05)
@@
 		)
 		(fp_line
-			(start 2.45 1.12)
-			(end -2.45 1.12)
+			(start -2.45 1.12)
+			(end -2.45 -1.12)
 			(stroke
 				(width 0.05)
@@
 		)
 		(fp_line
-			(start -2.45 1.12)
-			(end -2.45 -1.12)
+			(start -2.45 -1.12)
+			(end 2.45 -1.12)
 			(stroke
 				(width 0.05)
@@
 		)
 		(fp_line
-			(start 1.6 -0.8)
-			(end 1.6 0.8)
+			(start 1.6 0.8)
+			(end -1.6 0.8)
 			(stroke
 				(width 0.1)
@@
 		)
 		(fp_line
-			(start -1.6 -0.8)
-			(end 1.6 -0.8)
+			(start 1.6 -0.8)
+			(end 1.6 0.8)
 			(stroke
 				(width 0.1)
@@
 		)
 		(fp_line
-			(start 1.6 0.8)
-			(end -1.6 0.8)
+			(start -1.6 0.8)
+			(end -1.6 -0.8)
 			(stroke
 				(width 0.1)
@@
 		)
 		(fp_line
-			(start -1.6 0.8)
-			(end -1.6 -0.8)
+			(start -1.6 -0.8)
+			(end 1.6 -0.8)
 			(stroke
 				(width 0.1)
@@
 		)
 		(fp_text user "${REFERENCE}"
-			(at 0 0 90)
+			(at 0 0 360)
 			(layer "B.Fab")
 			(effects
@@
 		)
 		(pad "1" smd roundrect
-			(at -1.55 0 90)
+			(at -1.55 0 180)
 			(size 1.3 1.75)
 			(layers "B.Cu" "B.Paste" "B.Mask")
@@
 		)
 		(pad "2" smd roundrect
-			(at 1.55 0 90)
+			(at 1.55 0 180)
 			(size 1.3 1.75)
 			(layers "B.Cu" "B.Paste" "B.Mask")
@@
 	(footprint "Resistor_SMD:R_1206_3216Metric_Pad1.30x1.75mm_HandSolder"
 		(layer "B.Cu")
-		(at 141.5 100.95 90)
+		(at 139.25 103.45 90)
 		(descr "Resistor SMD 1206 (3216 Metric), square (rectangular) end terminal, IPC_7351 nominal with elongated pad for handsoldering. (Body size source: IPC-SM-782 page 72, https://www.pcb-3d.com/wordpress/wp-content/uploads/ipc-sm-782a_amendment_1_and_2.pdf), generated with kicad-footprint-generator")
 		(tags "resistor handsolder")
@@
 	)
 	(segment
-		(start 148.2 95)
+		(start 148.985126 98.25)
+		(end 149.025126 98.21)
+		(width 0.7)
+		(layer "B.Cu")
+		(net 7)
+	)
+	(segment
+		(start 149.025126 98.21)
+		(end 151.41 98.21)
+		(width 0.7)
+		(layer "B.Cu")
+		(net 7)
+	)
+	(segment
+		(start 136.16 94.41)
+		(end 140 98.25)
+		(width 0.7)
+		(layer "B.Cu")
+		(net 7)
+	)
+	(segment
+		(start 151.41 98.21)
 		(end 152 98.8)
 		(width 0.7)
@@
 	)
 	(segment
-		(start 136.16 90.2)
-		(end 140.96 95)
+		(start 140 98.25)
+		(end 148.985126 98.25)
 		(width 0.7)
 		(layer "B.Cu")
@@
 	)
 	(segment
-		(start 140.96 95)
-		(end 148.2 95)
+		(start 136.16 90.2)
+		(end 136.16 94.41)
 		(width 0.7)
 		(layer "B.Cu")
@@
 	)
 	(segment
-		(start 139.67 96.25)
-		(end 143 96.25)
-		(width 0.7)
-		(layer "B.Cu")
-		(net 24)
-	)
-	(segment
-		(start 143 96.25)
-		(end 146.25 99.5)
-		(width 0.7)
-		(layer "B.Cu")
-		(net 24)
-	)
-	(segment
-		(start 133.62 90.2)
-		(end 139.67 96.25)
-		(width 0.7)
-		(layer "B.Cu")
-		(net 24)
-	)
-	(segment
 		(start 121.15 82.1)
 		(end 118.16 79.11)
@@
 	)
 	(segment
-		(start 141.5 102.5)
-		(end 141.5 104.7)
-		(width 0.7)
-		(layer "B.Cu")
-		(net 33)
-	)
-	(segment
 		(start 148.288611 134.075)
 		(end 151.713611 137.5)
@@
 	)
 	(segment
-		(start 150.44 104.51)
-		(end 150.44 105.75)
-		(width 0.7)
-		(layer "B.Cu")
-		(net 34)
-	)
-	(segment
-		(start 156.95 116.2)
-		(end 158.75 116.2)
-		(width 0.7)
-		(layer "B.Cu")
-		(net 34)
-	)
-	(segment
-		(start 149.75 102.5)
-		(end 150.44 103.19)
-		(width 0.7)
-		(layer "B.Cu")
-		(net 34)
-	)
-	(segment
 		(start 158.75 116.2)
 		(end 161 116.2)
@@
 	)
 	(segment
-		(start 149.75 102.5)
-		(end 151.1 103.85)
-		(width 0.7)
-		(layer "B.Cu")
-		(net 34)
-	)
-	(segment
 		(start 161 116.2)
 		(end 167.9 123.1)
@@
 	)
 	(segment
-		(start 150.44 109.69)
-		(end 156.95 116.2)
-		(width 0.7)
-		(layer "B.Cu")
-		(net 34)
-	)
-	(segment
-		(start 150.44 103.19)
-		(end 150.44 105.75)
-		(width 0.7)
-		(layer "B.Cu")
-		(net 34)
-	)
-	(segment
-		(start 151.1 103.85)
-		(end 160.15 103.85)
-		(width 0.7)
-		(layer "B.Cu")
-		(net 34)
-	)
-	(segment
-		(start 150.44 105.75)
-		(end 150.44 109.69)
-		(width 0.7)
-		(layer "B.Cu")
-		(net 34)
-	)
-	(segment
-		(start 151.1 103.85)
-		(end 150.44 104.51)
-		(width 0.7)
-		(layer "B.Cu")
-		(net 34)
-	)
-	(segment
-		(start 160.15 103.85)
-		(end 161.75 102.25)
-		(width 0.7)
-		(layer "B.Cu")
-		(net 34)
-	)
-	(segment
 		(start 159.5 127.25)
 		(end 169.25 127.25)
@@
 	)
 	(segment
-		(start 141.5 99.4)
-		(end 143.2 101.1)
+		(start 144.25 100.162438)
+		(end 144.887438 99.525)
 		(width 0.7)
 		(layer "B.Cu")
@@
 	)
 	(segment
-		(start 147.6 101.1)
-		(end 148.74 99.96)
+		(start 144.25 102.25)
+		(end 144.25 100.162438)
 		(width 0.7)
 		(layer "B.Cu")
@@
 	)
 	(segment
-		(start 148.74 99.96)
+		(start 149.315 99.525)
 		(end 149.75 99.96)
 		(width 0.7)
@@
 	)
 	(segment
-		(start 143.2 101.1)
-		(end 147.6 101.1)
+		(start 139.25 101.9)
+		(end 140.325 102.975)
+		(width 0.7)
+		(layer "B.Cu")
+		(net 47)
+	)
+	(segment
+		(start 144.887438 99.525)
+		(end 149.315 99.525)
+		(width 0.7)
+		(layer "B.Cu")
+		(net 47)
+	)
+	(segment
+		(start 140.325 102.975)
+		(end 143.525 102.975)
+		(width 0.7)
+		(layer "B.Cu")
+		(net 47)
+	)
+	(segment
+		(start 143.525 102.975)
+		(end 144.25 102.25)
 		(width 0.7)
 		(layer "B.Cu")
@@
 	)
 	(segment
-		(start 159.21 98.76)
-		(end 159.21 102.25)
-		(width 0.7)
-		(layer "B.Cu")
-		(net 59)
-	)
-	(segment
-		(start 159 98.55)
-		(end 159.21 98.76)
-		(width 0.7)
-		(layer "B.Cu")
-		(net 59)
-	)
-	(segment
-		(start 146.3 106.6)
-		(end 146.3 102.65)
+		(start 145.75 106.05)
+		(end 146.3 106.6)
 		(width 0.7)
 		(layer "B.Cu")
@@
 	)
 	(segment
-		(start 146.3 102.65)
-		(end 146.25 102.6)
+		(start 145.75 102)
+		(end 145.75 106.05)
 		(width 0.7)
 		(layer "B.Cu")
